File: ledbase/Roco_44741/D99a.kicad_sch (KiCad schematic)
At the start: 0 parts

Commit message: add: ledbase Roco_44741
Other:
- title: Coach LED carrier PCB -> LED base: Roco #44741
Changed lines of the file:
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@@
 	(paper "A4")
 	(title_block
-		(title "Coach LED carrier PCB")
-		(date "2025-02-18")
-		(rev "0")
+		(title "LED base: Roco #44741")
+		(date "2025-10-19")
+		(rev "1")
 		(company "Frank Schumacher")
 		(comment 1 "D99a")
-		(comment 2 "Prototype 1")
+		(comment 2 "Prototype")
 	)
 	(sheet
