File: ledbase/Roco_44741/D99acpu.kicad_sch (KiCad schematic)
At the start: 21 parts, among them J1 Conn_01x01, J10 Conn_01x01, J11 Conn_01x01, J12 Conn_01x04, J13 Conn_01x06, J2 Conn_01x01, J3 Conn_01x01, J4 Conn_01x01, J5 Conn_02x10_Odd_Even, J6 Conn_01x01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

Commit message: add: ledbase Roco_44741
Other:
- title: Coach LED carrier PCB -> LED base: Roco #44741
Changed lines of the file:
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@@
 	(paper "A4")
 	(title_block
-		(title "Coach LED carrier PCB")
-		(date "2025-02-18")
-		(rev "0")
+		(title "LED base: Roco #44741")
+		(date "2025-10-19")
+		(rev "1")
 		(company "Frank Schumacher")
 		(comment 1 "D99a")
-		(comment 2 "Prototype 1")
+		(comment 2 "Prototype")
 	)
 	(text "SuperCap Solder Connect\n(must be 2.8V type)"
