File: D99.kicad_pcb (KiCad board)
At the start: 4 copper layers, 29.8 x 15 mm, 62 parts, among them IC1 TPS560430YFQDBVRQ1, IC2 NCP730BMT1500TBG, J1 Conn_02x10_Counter_Clockwise, Q1 BC847BDW1, Q2 BC857BDW1, Q3 BC847BDW1, U1 AVR-64DA48, U2 MAX40203AUK, U3 MCP1640BCH, U4 MAX40203AUK

Commit message: mod: ncap leakage resistor
Parts:
- added R29: 8.2k, Resistor_SMD:R_0402_1005Metric, F.Cu at (55.6, -70.2)
- D5, D6: footprint Diode_SMD:D_0603_1608Metric -> RTB:NSR20F40NXT5G
- L1: value 744029004 -> 4.7uH, 0.8A
- L2: value 744029004 -> 10uH, 1A
- moved R27 0.73 mm to (55.1, -71.6)
- moved D5 0.07 mm to (56.1, -66.6)
- renumbered Q3 to Q3B1
Connections:
- IC2 pad 2: (no net) -> unconnected-(IC2-NC/ADJ-Pad2)
- IC2 pad 5: (no net) -> unconnected-(IC2-NC/PG-Pad5)
- U1 pad 1: (no net) -> unconnected-(U1-PA5-Pad1)
- U1 pad 22: (no net) -> unconnected-(U1-PD2-Pad22)
- U1 pad 3: (no net) -> unconnected-(U1-PA7-Pad3)
- U1 pad 30: (no net) -> unconnected-(U1-PE0-Pad30)
- U1 pad 31: (no net) -> unconnected-(U1-PE1-Pad31)
- U1 pad 32: (no net) -> unconnected-(U1-PE2-Pad32)
- U1 pad 33: (no net) -> unconnected-(U1-PE3-Pad33)
- U1 pad 34: (no net) -> unconnected-(U1-PF0-Pad34)
- U1 pad 35: (no net) -> unconnected-(U1-PF1-Pad35)
- U1 pad 36: (no net) -> unconnected-(U1-PF2-Pad36)
- U1 pad 37: (no net) -> unconnected-(U1-PF3-Pad37)
- U1 pad 38: (no net) -> unconnected-(U1-PF4-Pad38)
- U1 pad 40: (no net) -> unconnected-(U1-PF6/~{RESET}-Pad40)
- U1 pad 45: (no net) -> unconnected-(U1-PA1-Pad45)
- U1 pad 8: (no net) -> unconnected-(U1-PB4-Pad8)
- U1 pad 9: (no net) -> unconnected-(U1-PB5-Pad9)
- U2 pad 4: (no net) -> unconnected-(U2-NC-Pad4)
- U4 pad 4: (no net) -> unconnected-(U4-NC-Pad4)
Routing:
- net VTRK: track 33.0 -> 35.6 mm
- net NCAP: track 5.66 -> 8.08 mm, vias 1 -> 3
- net Net-(IC2-OUT): track 4.57 -> 2.31 mm
- net LED.shcp: track 6.00 -> 7.15 mm, vias 0 -> 2
- net ~{LED.oe}: track 6.28 -> 5.76 mm
- net GND: vias 24 -> 25

Commit message: mod: refactoring
Parts:
- R29: value 8.2k -> 22k

Commit message: mod: refactoring
Parts:
- renumbered Q3B1 to Q3
Connections:
- Q3 pad 1: (no net) -> unconnected-(Q3A-E1-Pad1)
- Q3 pad 2: (no net) -> unconnected-(Q3A-B1-Pad2)
- Q3 pad 6: (no net) -> unconnected-(Q3A-C1-Pad6)
Changed lines of the file:
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@@
 	(net 46 "Net-(Q2A-B1)")
 	(net 47 "Net-(Q2A-C1)")
-	(net 48 "Net-(Q3B1B-B2)")
-	(net 49 "Net-(Q3B1B-C2)")
+	(net 48 "unconnected-(Q3A-B1-Pad2)")
+	(net 49 "unconnected-(Q3A-E1-Pad1)")
 	(net 50 "Net-(U1-PF5)")
 	(net 51 "Net-(U1-PD4)")
@@
 	(net 71 "unconnected-(U2-NC-Pad4)")
 	(net 72 "unconnected-(U4-NC-Pad4)")
+	(net 73 "Net-(Q3B-B2)")
+	(net 74 "Net-(Q3B-C2)")
+	(net 75 "unconnected-(Q3A-C1-Pad6)")
 	(footprint "Capacitor_SMD:C_0402_1005Metric"
 		(layer "F.Cu")
@@
 			(layers "F.Cu" "F.Mask" "F.Paste")
 			(roundrect_rratio 0.25)
-			(net 48 "Net-(Q3B1B-B2)")
+			(net 73 "Net-(Q3B-B2)")
 			(pintype "passive")
 		)
@@
 		(descr "SOT-363, SC-70-6, SC-88")
 		(tags "SOT-363 SC-70-6 SC-88")
-		(property "Reference" "Q3B1"
+		(property "Reference" "Q3"
 			(at 0 -2 90)
 			(layer "F.Fab")
@@
 			(layers "F.Cu" "F.Mask" "F.Paste")
 			(roundrect_rratio 0.25)
+			(net 49 "unconnected-(Q3A-E1-Pad1)")
+			(pinfunction "E1")
+			(pintype "passive+no_connect")
 		)
 		(pad "2" smd roundrect
@@
 			(layers "F.Cu" "F.Mask" "F.Paste")
 			(roundrect_rratio 0.25)
+			(net 48 "unconnected-(Q3A-B1-Pad2)")
+			(pinfunction "B1")
+			(pintype "input+no_connect")
 		)
 		(pad "3" smd roundrect
@@
 			(layers "F.Cu" "F.Mask" "F.Paste")
 			(roundrect_rratio 0.25)
-			(net 49 "Net-(Q3B1B-C2)")
+			(net 74 "Net-(Q3B-C2)")
 			(pinfunction "C2")
 			(pintype "passive")
@@
 			(layers "F.Cu" "F.Mask" "F.Paste")
 			(roundrect_rratio 0.25)
-			(net 48 "Net-(Q3B1B-B2)")
+			(net 73 "Net-(Q3B-B2)")
 			(pinfunction "B2")
 			(pintype "input")
@@
 			(layers "F.Cu" "F.Mask" "F.Paste")
 			(roundrect_rratio 0.25)
+			(net 75 "unconnected-(Q3A-C1-Pad6)")
+			(pinfunction "C1")
+			(pintype "passive+no_connect")
 		)
 		(embedded_fonts no)
@@
 			(layers "F.Cu" "F.Mask" "F.Paste")
 			(roundrect_rratio 0.25)
-			(net 49 "Net-(Q3B1B-C2)")
+			(net 74 "Net-(Q3B-C2)")
 			(pintype "passive")
 		)
@@
 		(net 47)
 	)
-	(via
-		(at 66.73 -71.73)
-		(size 0.5)
-		(drill 0.3)
-		(layers "F.Cu" "B.Cu")
-		(net 48)
-	)
-	(via
-		(at 71.61 -78.84)
-		(size 0.5)
-		(drill 0.3)
-		(layers "F.Cu" "B.Cu")
-		(net 48)
-	)
-	(segment
-		(start 67.290001 -72.290001)
-		(end 67.290001 -76.580001)
-		(width 0.1)
-		(layer "B.Cu")
-		(net 48)
-	)
-	(segment
-		(start 67.82 -77.11)
-		(end 71.34 -77.11)
-		(width 0.1)
-		(layer "B.Cu")
-		(net 48)
-	)
-	(segment
-		(start 66.73 -71.73)
-		(end 67.290001 -72.290001)
-		(width 0.1)
-		(layer "B.Cu")
-		(net 48)
-	)
-	(segment
-		(start 71.61 -77.38)
-		(end 71.61 -78.84)
-		(width 0.1)
-		(layer "B.Cu")
-		(net 48)
-	)
-	(segment
-		(start 71.34 -77.11)
-		(end 71.61 -77.38)
-		(width 0.1)
-		(layer "B.Cu")
-		(net 48)
-	)
-	(segment
-		(start 67.290001 -76.580001)
-		(end 67.82 -77.11)
-		(width 0.1)
-		(layer "B.Cu")
-		(net 48)
-	)
-	(segment
-		(start 72.26 -76.92)
-		(end 72.26 -75.795)
-		(width 0.2)
-		(layer "F.Cu")
-		(net 49)
-	)
-	(segment
-		(start 72.26 -75.795)
-		(end 72.545 -75.51)
-		(width 0.2)
-		(layer "F.Cu")
-		(net 49)
-	)
 	(segment
 		(start 55.27246 -75.34754)
@@
 		(net 54)
 	)
+	(via
+		(at 66.73 -71.73)
+		(size 0.5)
+		(drill 0.3)
+		(layers "F.Cu" "B.Cu")
+		(net 73)
+	)
+	(via
+		(at 71.61 -78.84)
+		(size 0.5)
+		(drill 0.3)
+		(layers "F.Cu" "B.Cu")
+		(net 73)
+	)
+	(segment
+		(start 67.290001 -72.290001)
+		(end 67.290001 -76.580001)
+		(width 0.1)
+		(layer "B.Cu")
+		(net 73)
+	)
+	(segment
+		(start 67.82 -77.11)
+		(end 71.34 -77.11)
+		(width 0.1)
+		(layer "B.Cu")
+		(net 73)
+	)
+	(segment
+		(start 66.73 -71.73)
+		(end 67.290001 -72.290001)
+		(width 0.1)
+		(layer "B.Cu")
+		(net 73)
+	)
+	(segment
+		(start 71.61 -77.38)
+		(end 71.61 -78.84)
+		(width 0.1)
+		(layer "B.Cu")
+		(net 73)
+	)
+	(segment
+		(start 71.34 -77.11)
+		(end 71.61 -77.38)
+		(width 0.1)
+		(layer "B.Cu")
+		(net 73)
+	)
+	(segment
+		(start 67.290001 -76.580001)
+		(end 67.82 -77.11)
+		(width 0.1)
+		(layer "B.Cu")
+		(net 73)
+	)
+	(segment
+		(start 72.26 -76.92)
+		(end 72.26 -75.795)
+		(width 0.2)
+		(layer "F.Cu")
+		(net 74)
+	)
+	(segment
+		(start 72.26 -75.795)
+		(end 72.545 -75.51)
+		(width 0.2)
+		(layer "F.Cu")
+		(net 74)
+	)
 	(zone
