File: D99cpu.kicad_sch (KiCad schematic)
At the start: 17 parts, among them J1 Conn_02x10_Counter_Clockwise, U1 AVR-64DA48

Commit message: initial
Other:
- note added: "Top View (J1 pins facing down)"
Changed lines of the file:
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@@
+		)
+	)
+	(text "Top View (J1 pins facing down)"
+		(exclude_from_sim no)
+		(at 221.234 133.604 0)
+		(effects
+			(font
+				(size 1.27 1.27)
+				(italic yes)
+			)
 		)
 	)

Commit message: mod: refactoring
Parts:
- C1, C2, C3: JLCPCB C1525 -> (none); LCSC Part # (none) -> C1525
- R1, R27: JLCPCB C25900 -> (none); LCSC Part # (none) -> C25900
- R10, R9: JLCPCB C25117 -> (none); LCSC Part # (none) -> C25117
- R2, R3: JLCPCB C25792 -> (none); LCSC Part # (none) -> C25792
- R4, R5, R8: JLCPCB C23162 -> (none); LCSC Part # (none) -> C23162
- U1: JLCPCB C3227399 -> (none); LCSC Part # (none) -> C3227399
Changed lines of the file:
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@@
 			)
 		)
-		(property "JLCPCB" "C1525"
+		(property "LCSC Part #" "C1525"
 			(at 113.03 46.99 0)
 			(effects
@@
 			)
 		)
-		(property "JLCPCB" "C1525"
+		(property "LCSC Part #" "C1525"
 			(at 118.11 46.99 0)
 			(effects
@@
 			)
 		)
-		(property "JLCPCB" "C3227399"
+		(property "LCSC Part #" "C3227399"
 			(at 88.9 87.63 0)
 			(effects
@@
 			)
 		)
-		(property "JLCPCB" "C1525"
+		(property "LCSC Part #" "C1525"
 			(at 107.95 46.99 0)
 			(effects
@@
 			)
 		)
-		(property "JLCPCB" "C25792"
+		(property "LCSC Part #" "C25792"
 			(at 63.5 113.03 90)
 			(effects
@@
 			)
 		)
-		(property "JLCPCB" "C23162"
+		(property "LCSC Part #" "C23162"
 			(at 232.41 45.72 90)
 			(effects
@@
 			)
 		)
-		(property "JLCPCB" "C23162"
+		(property "LCSC Part #" "C23162"
 			(at 222.25 54.61 90)
 			(effects
@@
 			)
 		)
-		(property "JLCPCB" "C23162"
+		(property "LCSC Part #" "C23162"
 			(at 222.25 59.69 90)
 			(effects
@@
 			)
 		)
-		(property "JLCPCB" "C25792"
+		(property "LCSC Part #" "C25792"
 			(at 63.5 107.95 90)
 			(effects
@@
 			)
 		)
-		(property "JLCPCB" "C25117"
+		(property "LCSC Part #" "C25117"
 			(at 236.22 102.87 90)
 			(effects
@@
 			)
 		)
-		(property "JLCPCB" "C25117"
+		(property "LCSC Part #" "C25117"
 			(at 236.22 105.41 90)
 			(effects
@@
 			)
 		)
-		(property "JLCPCB" "C25900"
+		(property "LCSC Part #" "C25900"
 			(at 63.5 74.93 90)
 			(effects
@@
 			)
 		)
-		(property "JLCPCB" "C25900"
+		(property "LCSC Part #" "C25900"
 			(at 114.3 58.42 90)
 			(effects
